Commit message: save

File: src/hexapod_description/urdf/robot.urdf (robot description, URDF)
Before this commit: robot hexapod, 19 links, 18 joints
Links:
- link base_link: geometry collision mesh filename=package://hexapod_description/meshes/body.stl; collision mesh filename=package://hexapod_description/meshes/bottom_cover.stl
- link foot_assembly: mass 0.635283 -> 0.633453; geometry collision mesh filename=package://hexapod_description/meshes/fixed_bracket.stl; collision mesh filename=package://hexapod_description/meshes/foot.stl
- link foot_assembly_2: mass 0.635283 -> 0.633453; geometry collision mesh filename=package://hexapod_description/meshes/fixed_bracket.stl; collision mesh filename=package://hexapod_description/meshes/foot.stl
- link foot_assembly_3: mass 0.635283 -> 0.633453; geometry collision mesh filename=package://hexapod_description/meshes/fixed_bracket.stl; collision mesh filename=package://hexapod_description/meshes/foot.stl
- link foot_assembly_4: mass 0.635283 -> 0.633453; geometry collision mesh filename=package://hexapod_description/meshes/fixed_bracket.stl; collision mesh filename=package://hexapod_description/meshes/foot.stl
- link foot_assembly_5: mass 0.635283 -> 0.633453; geometry collision mesh filename=package://hexapod_description/meshes/fixed_bracket.stl; collision mesh filename=package://hexapod_description/meshes/foot.stl
- link foot_assembly_6: mass 0.635283 -> 0.633453; geometry collision mesh filename=package://hexapod_description/meshes/fixed_bracket.stl; collision mesh filename=package://hexapod_description/meshes/foot.stl
- link hip_assembly: geometry collision mesh filename=package://hexapod_description/meshes/fixed_bracket.stl; collision mesh filename=package://hexapod_description/meshes/hip.stl
- link hip_assembly_2: geometry collision mesh filename=package://hexapod_description/meshes/fixed_bracket.stl; collision mesh filename=package://hexapod_description/meshes/hip.stl
- link hip_assembly_3: geometry collision mesh filename=package://hexapod_description/meshes/fixed_bracket.stl; collision mesh filename=package://hexapod_description/meshes/hip.stl
- link hip_assembly_4: geometry collision mesh filename=package://hexapod_description/meshes/fixed_bracket.stl; collision mesh filename=package://hexapod_description/meshes/hip.stl
- link hip_assembly_5: geometry collision mesh filename=package://hexapod_description/meshes/fixed_bracket.stl; collision mesh filename=package://hexapod_description/meshes/hip.stl
- link hip_assembly_6: geometry collision mesh filename=package://hexapod_description/meshes/fixed_bracket.stl; collision mesh filename=package://hexapod_description/meshes/hip.stl
- link ties_assembly: mass 0.589007 -> 0.589115; geometry collision mesh filename=package://hexapod_description/meshes/fixed_bracket.stl; collision mesh filename=package://hexapod_description/meshes/low_tie.stl
- link ties_assembly_2: mass 0.589007 -> 0.589115; geometry collision mesh filename=package://hexapod_description/meshes/fixed_bracket.stl; collision mesh filename=package://hexapod_description/meshes/low_tie.stl
- link ties_assembly_3: mass 0.589007 -> 0.589115; geometry collision mesh filename=package://hexapod_description/meshes/fixed_bracket.stl; collision mesh filename=package://hexapod_description/meshes/low_tie.stl
- link ties_assembly_4: mass 0.589007 -> 0.589115; geometry collision mesh filename=package://hexapod_description/meshes/fixed_bracket.stl; collision mesh filename=package://hexapod_description/meshes/low_tie.stl
- link ties_assembly_5: mass 0.589007 -> 0.589115; geometry collision mesh filename=package://hexapod_description/meshes/fixed_bracket.stl; collision mesh filename=package://hexapod_description/meshes/low_tie.stl
- link ties_assembly_6: mass 0.589007 -> 0.589115; geometry collision mesh filename=package://hexapod_description/meshes/fixed_bracket.stl; collision mesh filename=package://hexapod_description/meshes/low_tie.stl
Joints:
- joint foot_1: limit lower=-1.23378 upper=2.95501 effort=10 velocity=10 -> lower=-4.44089e-16 upper=4.18879 effort=10 velocity=10; origin xyz=0.188727 0.0341971 -0.000790548 rpy=7.80554e-16 1.23733e-15 2.45913 -> xyz=0.11535 0.153237 -0.000790548 rpy=4.79355e-16 9.68796e-16 1.97163
- joint foot_5: origin xyz=0.0850031 0.171935 -0.000790548 rpy=2.7886e-15 -1.77715e-15 2.22613 -> xyz=0.0850031 0.171935 -0.000790548 rpy=2.73845e-15 -1.75144e-15 2.22613
- joint hip_1: limit lower=-0.701492 upper=2.4401 effort=10 velocity=10 -> lower=-1.70171 upper=1.43988 effort=10 velocity=10; origin xyz=-0.242069 -0.318204 0.186418 rpy=4.41736e-16 -2.00843e-17 -0.523599 -> xyz=-0.479319 -0.438353 0.0695202 rpy=4.41736e-16 -2.00843e-17 -0.523599
- joint hip_2: origin xyz=-0.242069 -0.160413 0.186418 rpy=-2.65193e-15 4.96332e-16 -2.2469 -> xyz=-0.479319 -0.280563 0.0695202 rpy=-2.65193e-15 4.96332e-16 -2.2469
- joint hip_3: origin xyz=-0.37872 -0.0815178 0.187152 rpy=-2.0868e-15 1.31547e-15 -1.61555 -> xyz=-0.61597 -0.201668 0.0702537 rpy=-2.0868e-15 1.31547e-15 -1.61555
- joint hip_4: origin xyz=-0.51537 -0.160413 0.187152 rpy=-2.97536e-15 -4.73545e-16 -0.468195 -> xyz=-0.75262 -0.280563 0.0702537 rpy=-2.97536e-15 -4.73545e-16 -0.468195
- joint hip_5: origin xyz=-0.51537 -0.318204 0.125652 rpy=3.14159 1.60733e-15 0.64378 -> xyz=-0.75262 -0.438353 0.00875367 rpy=3.14159 1.60733e-15 0.64378
- joint hip_6: origin xyz=-0.37872 -0.397099 0.186418 rpy=1.19323e-15 -4.1531e-16 1.45631 -> xyz=-0.61597 -0.517249 0.0695202 rpy=1.19323e-15 -4.1531e-16 1.45631
- joint ties_1: limit lower=-1.92349 upper=1.56717 effort=10 velocity=10 -> lower=-2.66977 upper=0.820893 effort=10 velocity=10; origin xyz=0.0359262 -0.0907403 -0.0305 rpy=1.5708 5.59099e-16 -0.869304 -> xyz=0.0957704 -0.0187757 -0.0305 rpy=1.5708 1.85393e-15 0.130912

Commit message: save

File: src/hexapod_description/urdf/robot.urdf (robot description, URDF)
Before this commit: robot hexapod_description, 19 links, 18 joints
Links:
- link foot_assembly: mass 0.633453 -> 0.633745
- link foot_assembly_2: mass 0.633453 -> 0.633745
- link foot_assembly_3: mass 0.633453 -> 0.633745
- link foot_assembly_4: mass 0.633453 -> 0.633745
- link foot_assembly_5: mass 0.633453 -> 0.633745
- link foot_assembly_6: mass 0.633453 -> 0.633745
Joints:
- joint foot_1: limit lower=-4.44089e-16 upper=4.18879 effort=10 velocity=10 -> lower=-0.349066 upper=3.83972 effort=10 velocity=10; origin xyz=0.11535 0.153237 -0.000790548 rpy=4.79355e-16 9.68796e-16 1.97163 -> xyz=0.165999 0.0960821 -0.000790548 rpy=2.04167e-16 7.25873e-16 1.91986
- joint foot_2: limit lower=-0.0099805 upper=4.17881 effort=10 velocity=10 -> lower=-0.349066 upper=3.83972 effort=10 velocity=10; origin xyz=0.0723072 0.177648 -0.000790548 rpy=3.49334e-15 -4.3045e-15 2.24033 -> xyz=0.165999 0.0960821 -0.000790548 rpy=1.74534e-16 -7.20665e-17 1.91986
- joint foot_3: limit lower=-0.432463 upper=3.75633 effort=10 velocity=10 -> lower=-0.349066 upper=3.83972 effort=10 velocity=10; origin xyz=0.12627 0.144372 -0.000790548 rpy=1.20553e-14 8.1741e-16 2.33075 -> xyz=0.165999 0.0960821 -0.000790548 rpy=1.44039e-15 7.27652e-16 1.91986
- joint foot_4: limit lower=-0.324722 upper=3.86407 effort=10 velocity=10 -> lower=-0.349066 upper=3.83972 effort=10 velocity=10; origin xyz=0.112426 0.155395 -0.000790548 rpy=2.30727e-15 -2.8566e-15 2.31531 -> xyz=0.165999 0.0960821 -0.000790548 rpy=-6.20588e-15 -8.9332e-15 1.91986
- joint foot_5: limit lower=-0.0683837 upper=4.12041 effort=10 velocity=10 -> lower=-0.349066 upper=3.83972 effort=10 velocity=10; origin xyz=0.0850031 0.171935 -0.000790548 rpy=2.73845e-15 -1.75144e-15 2.22613 -> xyz=0.165999 0.0960821 -0.000790548 rpy=1.02679e-15 1.24004e-16 1.91986
- joint foot_6: limit lower=-0.605901 upper=3.58289 effort=10 velocity=10 -> lower=-0.349066 upper=3.83972 effort=10 velocity=10; origin xyz=0.172211 0.0844433 -0.000790548 rpy=-8.41938e-16 3.89144e-15 2.1079 -> xyz=0.165999 0.0960821 -0.000790548 rpy=-5.03397e-15 -1.50916e-14 1.91986
- joint hip_1: limit lower=-1.70171 upper=1.43988 effort=10 velocity=10 -> lower=-1.5708 upper=1.5708 effort=10 velocity=10; origin xyz=-0.479319 -0.438353 0.0695202 rpy=4.41736e-16 -2.00843e-17 -0.523599 -> xyz=-0.573739 -0.347776 0.386792 rpy=-3.98192e-14 -3.78648e-14 1.48353
- joint hip_2: limit lower=-1.94189 upper=1.19971 effort=10 velocity=10 -> lower=-1.5708 upper=1.5708 effort=10 velocity=10; origin xyz=-0.479319 -0.280563 0.0695202 rpy=-2.65193e-15 4.96332e-16 -2.2469 -> xyz=-0.716746 -0.414461 0.386792 rpy=5.13858e-14 -1.55159e-14 -0.610865
- joint hip_3: limit lower=-1.52605 upper=1.61555 effort=10 velocity=10 -> lower=-1.5708 upper=1.5708 effort=10 velocity=10; origin xyz=-0.61597 -0.201668 0.0702537 rpy=-2.0868e-15 1.31547e-15 -1.61555 -> xyz=-0.730498 -0.571652 0.387526 rpy=1.1508e-14 -5.35395e-14 0.436332
- joint hip_4: limit lower=-1.6262 upper=1.51539 effort=10 velocity=10 -> lower=-1.5708 upper=1.5708 effort=10 velocity=10; origin xyz=-0.75262 -0.280563 0.0702537 rpy=-2.97536e-15 -4.73545e-16 -0.468195 -> xyz=-0.601244 -0.662156 0.387526 rpy=-4.00013e-14 -3.73115e-14 1.48353
- joint hip_5: limit lower=-1.45061 upper=1.69098 effort=10 velocity=10 -> lower=-1.5708 upper=1.5708 effort=10 velocity=10; origin xyz=-0.75262 -0.438353 0.00875367 rpy=3.14159 1.60733e-15 0.64378 -> xyz=-0.458237 -0.595471 0.387526 rpy=5.12814e-14 -1.59069e-14 -0.610865
- joint hip_6: limit lower=-1.45631 upper=1.68529 effort=10 velocity=10 -> lower=-1.5708 upper=1.5708 effort=10 velocity=10; origin xyz=-0.61597 -0.517249 0.0695202 rpy=1.19323e-15 -4.1531e-16 1.45631 -> xyz=-0.444485 -0.438281 0.386792 rpy=-1.15359e-14 5.31115e-14 -2.70526
- joint ties_1: limit lower=-2.66977 upper=0.820893 effort=10 velocity=10 -> lower=-2.26893 upper=1.22173 effort=10 velocity=10; origin xyz=0.0957704 -0.0187757 -0.0305 rpy=1.5708 1.85393e-15 0.130912 -> xyz=0.0925 -0.0311167 -0.0305 rpy=1.5708 7.28949e-15 7.80449e-15
- joint ties_2: limit lower=-2.92848 upper=0.562177 effort=10 velocity=10 -> lower=-2.26893 upper=1.22173 effort=10 velocity=10; origin xyz=-0.0925 0.0311167 -0.0305 rpy=1.5708 -9.85323e-16 -3.14159 -> xyz=-0.0925 0.0311167 -0.0305 rpy=1.5708 -1.19807e-27 -3.14159
- joint ties_3: limit lower=-2.59641 upper=0.894244 effort=10 velocity=10 -> lower=-2.26893 upper=1.22173 effort=10 velocity=10; origin xyz=-0.0925 0.0311167 -0.0305 rpy=1.5708 -8.32667e-16 3.14159 -> xyz=-0.0925 0.0311167 -0.0305 rpy=1.5708 -3.15544e-29 -3.14159
- joint ties_4: limit lower=-2.68872 upper=0.801941 effort=10 velocity=10 -> lower=-2.26893 upper=1.22173 effort=10 velocity=10; origin xyz=-0.0925 0.0311167 -0.0305 rpy=1.5708 -9.71445e-17 -3.14159 -> xyz=-0.0925 0.0311167 -0.0305 rpy=1.5708 -3.33266e-16 -3.14159
- joint ties_5: limit lower=-2.85588 upper=0.634779 effort=10 velocity=10 -> lower=-2.26893 upper=1.22173 effort=10 velocity=10; origin xyz=-0.0925 -0.0311167 -0.0305 rpy=-1.5708 -1.38778e-16 3.14159 -> xyz=0.0925 -0.0311167 -0.0305 rpy=1.5708 -7.65103e-16 -1.70903e-16
- joint ties_6: limit lower=-2.20013 upper=1.29053 effort=10 velocity=10 -> lower=-2.26893 upper=1.22173 effort=10 velocity=10; origin xyz=-0.0925 0.0311167 -0.0305 rpy=1.5708 -1.18004e-15 -3.14159 -> xyz=-0.0925 0.0311167 -0.0305 rpy=1.5708 1.35775e-15 3.14159

Commit message: save

File: src/hexapod_description/urdf/robot.urdf (robot description, URDF)
Before this commit: robot hexapod_description, 19 links, 18 joints
Links:
- link base_link: mass 2.24777 -> 2.26596; geometry collision mesh filename=package://hexapod_description/meshes/body_brain.stl; collision mesh filename=package://hexapod_description/meshes/body_power.stl
Joints:
- joint foot_1: origin xyz=0.165999 0.0960821 -0.000790548 rpy=2.04167e-16 7.25873e-16 1.91986 -> xyz=0.165999 0.0960821 -0.000790548 rpy=1.05854e-17 1.13313e-14 1.91986
- joint foot_2: origin xyz=0.165999 0.0960821 -0.000790548 rpy=1.74534e-16 -7.20665e-17 1.91986 -> xyz=0.165999 0.0960821 -0.000790548 rpy=-1.18413e-16 1.60207e-15 1.91986
- joint foot_3: origin xyz=0.165999 0.0960821 -0.000790548 rpy=1.44039e-15 7.27652e-16 1.91986 -> xyz=0.165999 0.0960821 -0.000790548 rpy=-2.99398e-16 -1.37685e-16 1.91986
- joint foot_4: origin xyz=0.165999 0.0960821 -0.000790548 rpy=-6.20588e-15 -8.9332e-15 1.91986 -> xyz=0.165999 0.0960821 -0.000790548 rpy=1.4637e-15 1.68038e-16 1.91986
- joint foot_5: origin xyz=0.165999 0.0960821 -0.000790548 rpy=1.02679e-15 1.24004e-16 1.91986 -> xyz=0.165999 0.0960821 -0.000790548 rpy=-3.9985e-15 -5.62892e-15 1.91986
- joint foot_6: origin xyz=0.165999 0.0960821 -0.000790548 rpy=-5.03397e-15 -1.50916e-14 1.91986 -> xyz=0.165999 0.0960821 -0.000790548 rpy=-6.52802e-17 -1.18702e-16 1.91986
- joint hip_1: origin xyz=-0.573739 -0.347776 0.386792 rpy=-3.98192e-14 -3.78648e-14 1.48353 -> xyz=0.0202915 0.148301 0.0272372 rpy=-3.93428e-14 -3.97183e-14 1.48353
- joint hip_2: origin xyz=-0.716746 -0.414461 0.386792 rpy=5.13858e-14 -1.55159e-14 -0.610865 -> xyz=0.144817 0.0611074 0.0272372 rpy=-1.39309e-14 5.38714e-14 -2.70526
- joint hip_3: origin xyz=-0.730498 -0.571652 0.387526 rpy=1.1508e-14 -5.35395e-14 0.436332 -> xyz=0.131567 -0.0903312 0.0279706 rpy=-5.21664e-14 1.54145e-14 2.53073
- joint hip_4: origin xyz=-0.601244 -0.662156 0.387526 rpy=-4.00013e-14 -3.73115e-14 1.48353 -> xyz=-0.0062068 -0.154576 0.0279706 rpy=-3.88964e-14 -3.72989e-14 1.48353
- joint hip_5: origin xyz=-0.458237 -0.595471 0.387526 rpy=5.12814e-14 -1.59069e-14 -0.610865 -> xyz=-0.130732 -0.0673829 0.0279706 rpy=-1.23219e-14 5.33622e-14 -2.70526
- joint hip_6: origin xyz=-0.444485 -0.438281 0.386792 rpy=-1.15359e-14 5.31115e-14 -2.70526 -> xyz=-0.117483 0.0840557 0.0272372 rpy=5.19508e-14 -1.48406e-14 -0.610865
- joint ties_1: origin xyz=0.0925 -0.0311167 -0.0305 rpy=1.5708 7.28949e-15 7.80449e-15 -> xyz=0.0925 -0.0311167 -0.0305 rpy=1.5708 3.25123e-15 3.22165e-16
- joint ties_2: origin xyz=-0.0925 0.0311167 -0.0305 rpy=1.5708 -1.19807e-27 -3.14159 -> xyz=-0.0925 0.0311167 -0.0305 rpy=1.5708 3.50154e-15 3.14159
- joint ties_3: origin xyz=-0.0925 0.0311167 -0.0305 rpy=1.5708 -3.15544e-29 -3.14159 -> xyz=-0.0925 0.0311167 -0.0305 rpy=1.5708 -8.53508e-17 -3.14159
- joint ties_4: origin xyz=-0.0925 0.0311167 -0.0305 rpy=1.5708 -3.33266e-16 -3.14159 -> xyz=-0.0925 0.0311167 -0.0305 rpy=1.5708 -1.87979e-15 -3.14159
- joint ties_5: origin xyz=0.0925 -0.0311167 -0.0305 rpy=1.5708 -7.65103e-16 -1.70903e-16 -> xyz=0.0925 -0.0311167 -0.0305 rpy=1.5708 2.88289e-16 1.53604e-15
- joint ties_6: origin xyz=-0.0925 0.0311167 -0.0305 rpy=1.5708 1.35775e-15 3.14159 -> xyz=-0.0925 0.0311167 -0.0305 rpy=1.5708 1.0413e-28 3.14159
