Commit message: save

File: hexapod_py/platform/simulation/robot.urdf (robot description, URDF)
Before this commit: robot C:\Users\gata2\OneDrive\Documents\hexapod\hexapod_py\simulation, 19 links, 18 joints
Links:
- link base_link: mass 2.53298 -> 2.35252; geometry collision mesh filename=package://meshes\body_brain.stl; collision mesh filename=package://meshes\body_power.stl
- link foot_assembly: mass 0.633745 -> 0.628062
- link foot_assembly_2: mass 0.633745 -> 0.628062
- link foot_assembly_3: mass 0.633745 -> 0.628062
- link foot_assembly_4: mass 0.633745 -> 0.628062
- link foot_assembly_5: mass 0.633745 -> 0.628062
- link foot_assembly_6: mass 0.633745 -> 0.628062
- link hip_assembly: mass 0.365356 -> 0.38056
- link hip_assembly_2: mass 0.365356 -> 0.38056
- link hip_assembly_3: mass 0.365356 -> 0.38056
- link hip_assembly_4: mass 0.365356 -> 0.38056
- link hip_assembly_5: mass 0.365356 -> 0.38056
- link hip_assembly_6: mass 0.365356 -> 0.38056
- link ties_assembly: mass 0.589115 -> 0.581468
- link ties_assembly_2: mass 0.589115 -> 0.581468
- link ties_assembly_3: mass 0.589115 -> 0.581468
- link ties_assembly_4: mass 0.589115 -> 0.581468
- link ties_assembly_5: mass 0.589115 -> 0.581468
- link ties_assembly_6: mass 0.589115 -> 0.581468
Joints:
- joint foot_1: origin xyz=0.1918 0.000210323 -0.000790548 rpy=-1.66622e-14 -3.69666e-15 3.14159 -> xyz=0.1918 0.000117091 -0.00186036 rpy=-1.83367e-15 -1.8597e-15 3.14159
- joint foot_2: origin xyz=0.1918 0.000210323 -0.000790548 rpy=2.57504e-15 -5.91728e-15 3.14159 -> xyz=0.1918 0.000117091 -0.00186036 rpy=-6.33457e-15 -1.83953e-14 3.14159
- joint foot_3: origin xyz=0.1918 0.000210323 -0.000790548 rpy=1.68416e-15 -9.61937e-17 3.14159 -> xyz=0.1918 0.000117091 -0.00186036 rpy=1.26193e-15 -1.75295e-15 -3.14159
- joint foot_4: origin xyz=0.1918 0.000210323 -0.000790548 rpy=-1.34033e-15 3.08383e-16 -3.14159 -> xyz=0.1918 0.000117091 -0.00186036 rpy=-1.51606e-14 -1.33155e-14 -3.14159
- joint foot_5: origin xyz=0.1918 0.000210323 -0.000790548 rpy=3.64523e-14 3.95047e-14 3.14159 -> xyz=0.1918 0.000117091 -0.00186036 rpy=3.30023e-17 1.82639e-15 3.14159
- joint foot_6: origin xyz=0.1918 0.000210323 -0.000790548 rpy=-1.79782e-15 2.47828e-15 -3.14159 -> xyz=0.1918 0.000117091 -0.00186036 rpy=2.27858e-15 -2.06207e-16 -3.14159
- joint hip_1: origin xyz=0.138321 0.0680226 0.0134908 rpy=-2.3989e-14 -2.8749e-14 0.436332 -> xyz=0.142873 0.0479466 0.0166947 rpy=-2.41992e-14 -2.85159e-14 0.436332
- joint hip_2: origin xyz=0.125071 -0.083416 0.0134908 rpy=-7.92838e-15 3.38805e-14 2.53073 -> xyz=0.129624 -0.103492 0.0166947 rpy=-1.34586e-14 3.21607e-14 2.53073
- joint hip_3: origin xyz=-0.0127028 -0.147661 0.0142242 rpy=3.23352e-14 -8.74693e-15 -1.65806 -> xyz=-0.00815056 -0.167737 0.0174281 rpy=7.71669e-15 -8.74693e-15 -1.65806
- joint hip_4: origin xyz=-0.137228 -0.0604678 0.0142242 rpy=2.50355e-14 2.47371e-14 -2.70526 -> xyz=-0.132676 -0.0805438 0.0174281 rpy=2.48412e-14 2.47371e-14 -2.70526
- joint hip_5: origin xyz=-0.123979 0.0909708 0.0142242 rpy=7.95355e-15 3.42754e-14 2.53073 -> xyz=-0.119426 0.0708948 0.0174281 rpy=-4.50694e-15 3.38573e-14 2.53073
- joint hip_6: origin xyz=0.0137956 0.155216 0.0134908 rpy=-1.77288e-14 1.38591e-15 1.48353 -> xyz=0.0183478 0.13514 0.0166947 rpy=-3.01521e-14 7.87813e-15 1.48353
- joint ties_1: origin xyz=0.0925 -0.0311167 -0.0305 rpy=1.5708 4.45935e-15 2.48483e-12 -> xyz=0.0925 -0.0311167 -0.0305 rpy=1.5708 3.75284e-15 1.25724e-15
- joint ties_2: origin xyz=-0.0925 0.0311167 -0.0305 rpy=1.5708 -8.55001e-16 3.14159 -> xyz=-0.0925 0.0311167 -0.0305 rpy=1.5708 -2.48572e-15 3.14159
- joint ties_3: origin xyz=0.0925 -0.0311167 -0.0305 rpy=1.5708 9.22412e-17 2.50162e-12 -> xyz=0.0925 -0.0311167 -0.0305 rpy=1.5708 -2.74219e-14 9.4696e-15
- joint ties_4: origin xyz=0.0925 -0.0311167 -0.0305 rpy=1.5708 6.76543e-16 2.49947e-12 -> xyz=0.0925 -0.0311167 -0.0305 rpy=1.5708 6.85694e-16 -2.44517e-16
- joint ties_5: origin xyz=0.0925 -0.0311167 -0.0305 rpy=1.5708 5.4278e-16 2.49541e-12 -> xyz=0.0925 -0.0311167 -0.0305 rpy=1.5708 7.61127e-15 1.9026e-16
- joint ties_6: origin xyz=0.0925 -0.0311167 -0.0305 rpy=1.5708 7.98949e-15 2.49698e-12 -> xyz=0.0925 -0.0311167 -0.0305 rpy=1.5708 3.18423e-14 5.08286e-14
